File: PowerBox_PCB/BMS.kicad_sch (KiCad schematic)
At the start: 12 parts

Commit message: .
Changed lines of the file:
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@@
 		(lib_id "Custom_Symbols:0.1uF")
 		(at 144.78 80.01 0)
+		(mirror y)
 		(unit 1)
 		(body_style 1)
@@
 		(in_pos_files yes)
 		(dnp no)
-		(fields_autoplaced yes)
 		(property "Reference" "C21"
-			(at 148.59 78.7399 0)
+			(at 140.97 78.7399 0)
 			(show_name no)
 			(do_not_autoplace no)
@@
 		)
 		(property "Value" "0.1uF"
-			(at 148.59 81.2799 0)
+			(at 140.97 81.2799 0)
 			(show_name no)
 			(do_not_autoplace no)
@@
 		(lib_id "Custom_Symbols:0.1uF")
 		(at 144.78 100.33 0)
+		(mirror y)
 		(unit 1)
 		(body_style 1)
@@
 		(in_pos_files yes)
 		(dnp no)
-		(fields_autoplaced yes)
 		(property "Reference" "C22"
-			(at 148.59 99.0599 0)
+			(at 140.97 99.0599 0)
 			(show_name no)
 			(do_not_autoplace no)
@@
 		)
 		(property "Value" "0.1uF"
-			(at 148.59 101.5999 0)
+			(at 140.97 101.5999 0)
 			(show_name no)
 			(do_not_autoplace no)

Commit message: fix bom
bom
Parts:
- U11, U15: value (none) -> DW01A
- U13, U14, U16, U17: value (none) -> AO3400A
Changed lines of the file:
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@@
 		(in_pos_files yes)
 		(dnp no)
-		(fields_autoplaced yes)
 		(property "Reference" "U13"
-			(at 165.1 90.17 90)
-			(show_name no)
-			(do_not_autoplace no)
-			(effects
-				(font
-					(size 1.27 1.27)
-				)
-			)
-		)
-		(property "Value" ""
-			(at 165.1 86.36 0)
+			(at 165.1 89.408 90)
+			(show_name no)
+			(do_not_autoplace no)
+			(effects
+				(font
+					(size 1.27 1.27)
+				)
+			)
+		)
+		(property "Value" "AO3400A"
+			(at 165.1 91.186 90)
 			(show_name no)
 			(do_not_autoplace no)
@@
 		(in_pos_files yes)
 		(dnp no)
-		(fields_autoplaced yes)
 		(property "Reference" "U16"
 			(at 165.1 110.49 90)
@@
 			)
 		)
-		(property "Value" ""
-			(at 165.1 106.68 0)
+		(property "Value" "AO3400A"
+			(at 165.1 112.776 90)
 			(show_name no)
 			(do_not_autoplace no)
@@
 			)
 		)
-		(property "Value" ""
-			(at 157.48 96.52 0)
+		(property "Value" "DW01A"
+			(at 157.48 101.6 0)
 			(show_name no)
 			(do_not_autoplace no)
@@
 		(dnp no)
 		(property "Reference" "U14"
-			(at 175.26 90.17 90)
-			(show_name no)
-			(do_not_autoplace no)
-			(effects
-				(font
-					(size 1.27 1.27)
-				)
-			)
-		)
-		(property "Value" ""
-			(at 175.26 86.36 0)
+			(at 175.26 89.408 90)
+			(show_name no)
+			(do_not_autoplace no)
+			(effects
+				(font
+					(size 1.27 1.27)
+				)
+			)
+		)
+		(property "Value" "AO3400A"
+			(at 175.26 91.44 90)
 			(show_name no)
 			(do_not_autoplace no)
@@
 			)
 		)
-		(property "Value" ""
-			(at 157.48 76.2 0)
+		(property "Value" "DW01A"
+			(at 157.48 81.28 0)
 			(show_name no)
 			(do_not_autoplace no)
@@
 			)
 		)
-		(property "Value" ""
-			(at 175.26 106.68 0)
-			(show_name no)
-			(do_not_autoplace no)
+		(property "Value" "AO3400A"
+			(at 175.26 112.522 90)
+			(show_name no)
+			(do_not_autoplace no)
