File: PowerBox_PCB/Ideal_Diode.kicad_sch (KiCad schematic)
At the start: 5 parts

Commit message: fix bom
bom
Parts:
- U2, U4: value (none) -> MMBT3906LT1G
- U3: value (none) -> DMP6023LE-13
Changed lines of the file:
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@@
 			)
 		)
-		(property "Value" ""
-			(at 101.6 88.9 0)
+		(property "Value" "MMBT3906LT1G"
+			(at 87.884 88.9 0)
 			(show_name no)
 			(do_not_autoplace no)
@@
 			)
 		)
-		(property "Value" ""
-			(at 121.92 88.9 0)
+		(property "Value" "MMBT3906LT1G"
+			(at 135.636 88.9 0)
 			(show_name no)
 			(do_not_autoplace no)
@@
 		(in_pos_files yes)
 		(dnp no)
-		(fields_autoplaced yes)
 		(property "Reference" "U3"
 			(at 111.76 71.12 90)
@@
 			)
 		)
-		(property "Value" ""
-			(at 111.76 74.93 0)
-			(show_name no)
-			(do_not_autoplace no)
+		(property "Value" "DMP6023LE-13"
+			(at 111.76 67.818 90)
+			(show_name no)
+			(do_not_autoplace no)
