File: PowerBox_PCB/TPS54620_Buck.kicad_sch (KiCad schematic)
At the start: 17 parts

Commit message: .
Changed lines of the file:
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@@
 		(lib_id "Buck_TPS54620:30pF_Cap_0805")
 		(at 119.38 115.57 0)
-		(unit 1)
-		(body_style 1)
-		(exclude_from_sim no)
-		(in_bom yes)
-		(on_board yes)
-		(in_pos_files yes)
-		(dnp no)
-		(fields_autoplaced yes)
+		(mirror y)
+		(unit 1)
+		(body_style 1)
+		(exclude_from_sim no)
+		(in_bom yes)
+		(on_board yes)
+		(in_pos_files yes)
+		(dnp no)
 		(property "Reference" "C8"
-			(at 123.19 114.2999 0)
+			(at 116.586 115.57 0)
 			(show_name no)
 			(do_not_autoplace no)
@@
 		)
 		(property "Value" "30pF"
-			(at 123.19 116.8399 0)
+			(at 116.84 118.364 0)
 			(show_name no)
 			(do_not_autoplace no)
@@
 		(lib_id "Buck_TPS54620:53.6kΩ_Res_0805")
 		(at 114.3 106.68 0)
-		(unit 1)
-		(body_style 1)
-		(exclude_from_sim no)
-		(in_bom yes)
-		(on_board yes)
-		(in_pos_files yes)
-		(dnp no)
-		(fields_autoplaced yes)
+		(mirror y)
+		(unit 1)
+		(body_style 1)
+		(exclude_from_sim no)
+		(in_bom yes)
+		(on_board yes)
+		(in_pos_files yes)
+		(dnp no)
 		(property "Reference" "R5"
-			(at 116.84 105.4099 0)
+			(at 112.522 105.41 0)
 			(show_name no)
 			(do_not_autoplace no)
@@
 		)
 		(property "Value" "53.6kΩ"
-			(at 116.84 107.9499 0)
+			(at 112.522 107.95 0)
 			(show_name no)
 			(do_not_autoplace no)
@@
 		(in_pos_files yes)
 		(dnp no)
-		(fields_autoplaced yes)
 		(property "Reference" "C7"
-			(at 120.65 90.17 90)
+			(at 120.65 94.488 90)
 			(show_name no)
 			(do_not_autoplace no)
@@
 		)
 		(property "Value" "2.2uF"
-			(at 120.65 92.71 90)
+			(at 124.714 99.314 90)
 			(show_name no)
 			(do_not_autoplace no)
@@
 		(in_pos_files yes)
 		(dnp no)
-		(fields_autoplaced yes)
 		(property "Reference" "C5"
-			(at 85.09 91.4399 0)
+			(at 80.264 89.408 90)
 			(show_name no)
 			(do_not_autoplace no)
@@
 		)
 		(property "Value" "4.7uF"
-			(at 85.09 93.9799 0)
+			(at 82.296 89.408 90)
 			(show_name no)
 			(do_not_autoplace no)
@@
 		(in_pos_files yes)
 		(dnp no)
-		(fields_autoplaced yes)
 		(property "Reference" "C6"
-			(at 80.01 91.4399 0)
+			(at 75.184 89.408 90)
 			(show_name no)
 			(do_not_autoplace no)
@@
 		)
 		(property "Value" "4.7uF"
-			(at 80.01 93.9799 0)
+			(at 77.216 89.408 90)
 			(show_name no)
 			(do_not_autoplace no)
@@
 		(in_pos_files yes)
 		(dnp no)
-		(fields_autoplaced yes)
 		(property "Reference" "C4"
-			(at 90.17 91.4399 0)
+			(at 85.344 89.408 90)
 			(show_name no)
 			(do_not_autoplace no)
@@
 		)
 		(property "Value" "4.7uF"
-			(at 90.17 93.9799 0)
+			(at 87.376 89.408 90)
 			(show_name no)
 			(do_not_autoplace no)
@@
 		(in_pos_files yes)
 		(dnp no)
-		(fields_autoplaced yes)
 		(property "Reference" "C3"
-			(at 97.79 91.4399 0)
+			(at 92.964 89.662 90)
 			(show_name no)
 			(do_not_autoplace no)
@@
 		)
 		(property "Value" "4.7uF"
-			(at 97.79 93.9799 0)
+			(at 95.25 89.662 90)
 			(show_name no)
 			(do_not_autoplace no)
@@
 		(in_pos_files yes)
 		(dnp no)
-		(fields_autoplaced yes)
 		(property "Reference" "#PWR04"
 			(at 116.84 104.14 0)
@@
 		)
 		(property "Value" "GND"
-			(at 116.84 102.87 0)
+			(at 116.84 101.6 0)
 			(show_name no)
 			(do_not_autoplace no)
@@
 		(in_pos_files yes)
 		(dnp no)
-		(fields_autoplaced yes)
 		(property "Reference" "#PWR03"
 			(at 114.3 116.84 0)
@@
 		)
 		(property "Value" "GND"
-			(at 114.3 115.57 0)
+			(at 114.3 113.792 0)
 			(show_name no)
 			(do_not_autoplace no)
@@
 		(in_pos_files yes)
 		(dnp no)
-		(fields_autoplaced yes)
 		(property "Reference" "C1"
-			(at 158.75 80.01 90)
+			(at 163.83 86.868 90)
 			(show_name no)
 			(do_not_autoplace no)
@@
 		)
 		(property "Value" "100nf"
-			(at 158.75 82.55 90)
+			(at 162.814 89.154 90)
 			(show_name no)
 			(do_not_autoplace no)
@@
 		(lib_id "Buck_TPS54620:52.3kΩ_Res_0805")
 		(at 176.53 88.9 0)
-		(unit 1)
-		(body_style 1)
-		(exclude_from_sim no)
-		(in_bom yes)
-		(on_board yes)
-		(in_pos_files yes)
-		(dnp no)
-		(fields_autoplaced yes)
+		(mirror y)
+		(unit 1)
+		(body_style 1)
+		(exclude_from_sim no)
+		(in_bom yes)
+		(on_board yes)
+		(in_pos_files yes)
+		(dnp no)
 		(property "Reference" "R1"
-			(at 179.07 87.6299 0)
+			(at 173.99 87.6299 0)
 			(show_name no)
 			(do_not_autoplace no)
@@
 		)
 		(property "Value" "52.3kΩ"
-			(at 179.07 90.1699 0)
-			(show_name no)
-			(do_not_autoplace no)
+			(at 173.99 90.1699 0)
+			(show_name no)
+			(do_not_autoplace no)

Commit message: fix bom
bom
Parts:
- U1: value (none) -> TPS54620
Changed lines of the file:
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@@
 			)
 		)
-		(property "Value" ""
+		(property "Value" "TPS54620"
 			(at 139.7 95.25 0)
 			(show_name no)

Commit message: Changed HUSB238 to CH221K
HUSB238 Went out of stock so changed to CH221K
Parts:
- removed C2: 47uF, Capacitor_SMD:C_0805_2012Metric_Pad1.18x1.45mm_HandSolder, symbol Buck_TPS54620:47uF_Cap_0805
- added C19: 47uF, Capacitor_SMD:C_1210_3225Metric_Pad1.33x2.70mm_HandSolder, symbol Buck_TPS54620:47uF_Cap_1210
- L1: footprint Buck_TPS54620:3.3uH_SMD,10x10mm -> Buck_TPS54620:IND-SMD_L8.5-W8.0_PSPMAA0803H-330M-ANP
Connections:
- net GND: now also C19.2
- net VOUT_BUCK: now also C19.1
Changed lines of the file:
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@@
 			)
 		)
-		(property "Footprint" "Buck_TPS54620:3.3uH_SMD,10x10mm"
+		(property "Footprint" "Buck_TPS54620:IND-SMD_L8.5-W8.0_PSPMAA0803H-330M-ANP"
 			(at 168.91 82.55 0)
 			(hide yes)
@@
 	)
 	(symbol
-		(lib_id "Buck_TPS54620:47uF_Cap_0805")
-		(at 185.42 92.71 0)
-		(unit 1)
-		(body_style 1)
-		(exclude_from_sim no)
-		(in_bom yes)
-		(on_board yes)
-		(in_pos_files yes)
-		(dnp no)
-		(fields_autoplaced yes)
-		(property "Reference" "C2"
-			(at 189.23 91.4399 0)
-			(show_name no)
-			(do_not_autoplace no)
-			(effects
-				(font
-					(size 1.27 1.27)
-				)
-				(justify left)
-			)
-		)
-		(property "Value" "47uF"
-			(at 189.23 93.9799 0)
-			(show_name no)
-			(do_not_autoplace no)
-			(effects
-				(font
-					(size 1.27 1.27)
-				)
-				(justify left)
-			)
-		)
-		(property "Footprint" "Capacitor_SMD:C_0805_2012Metric_Pad1.18x1.45mm_HandSolder"
-			(at 185.42 92.71 0)
-			(hide yes)
-			(show_name no)
-			(do_not_autoplace no)
-			(effects
-				(font
-					(size 1.27 1.27)
-				)
-			)
-		)
-		(property "Datasheet" ""
-			(at 185.42 92.71 0)
-			(hide yes)
-			(show_name no)
-			(do_not_autoplace no)
-			(effects
-				(font
-					(size 1.27 1.27)
-				)
-			)
-		)
-		(property "Description" ""
-			(at 185.42 92.71 0)
-			(hide yes)
-			(show_name no)
-			(do_not_autoplace no)
-			(effects
-				(font
-					(size 1.27 1.27)
-				)
-			)
-		)
-		(pin "2"
-		)
-		(pin "1"
-		)
-		(instances
-			(project "PowerBox_PCB"
-				(path "/b0254e12-8cc0-427f-8cea-8f6ec8f66525/95341a3d-fa0d-4381-83e3-fd64358ddeb4"
-					(reference "C18")
-					(unit 1)
-				)
-				(path "/b0254e12-8cc0-427f-8cea-8f6ec8f66525/ba8d25d8-5959-48f3-8926-1c1b4d717b71"
-					(reference "C2")
-					(unit 1)
-				)
-			)
-		)
-	)
-	(symbol
 		(lib_id "power:GND")
 		(at 154.94 107.95 0)
@@
 					(unit 1)
 				)
+			)
+		)
+	)
+	(symbol
+		(lib_id "Buck_TPS54620:47uF_Cap_1210")
+		(at 185.42 92.71 0)
+		(unit 1)
+		(body_style 1)
+		(exclude_from_sim no)
+		(in_bom yes)
+		(on_board yes)
+		(in_pos_files yes)
+		(dnp no)
+		(fields_autoplaced yes)
+		(property "Reference" "C19"
+			(at 189.23 91.4399 0)
+			(show_name no)
+			(do_not_autoplace no)
+			(effects
+				(font
+					(size 1.27 1.27)
+				)
+				(justify left)
+			)
+		)
+		(property "Value" "47uF"
+			(at 189.23 93.9799 0)
+			(show_name no)
+			(do_not_autoplace no)
+			(effects
+				(font
+					(size 1.27 1.27)
+				)
+				(justify left)
+			)
+		)
+		(property "Footprint" "Capacitor_SMD:C_1210_3225Metric_Pad1.33x2.70mm_HandSolder"
+			(at 185.42 92.71 0)
+			(hide yes)
+			(show_name no)
+			(do_not_autoplace no)
+			(effects
+				(font
+					(size 1.27 1.27)
+				)
+			)
+		)
+		(property "Datasheet" ""
+			(at 185.42 92.71 0)
+			(hide yes)
+			(show_name no)
+			(do_not_autoplace no)
+			(effects
+				(font
+					(size 1.27 1.27)
+				)
+			)
+		)
+		(property "Description" ""
+			(at 185.42 92.71 0)
+			(hide yes)
+			(show_name no)
+			(do_not_autoplace no)
+			(effects
+				(font
+					(size 1.27 1.27)
+				)
+			)
+		)
+		(pin "2"
+		)
+		(pin "1"
+		)
+		(instances
+			(project "PowerBox_PCB"
+				(path "/b0254e12-8cc0-427f-8cea-8f6ec8f66525/95341a3d-fa0d-4381-83e3-fd64358ddeb4"
+					(reference "C23")
+					(unit 1)
+				)
+				(path "/b0254e12-8cc0-427f-8cea-8f6ec8f66525/ba8d25d8-5959-48f3-8926-1c1b4d717b71"
+					(reference "C19")
+					(unit 1)
+				)
