File: PowerBox_PCB/Batt Charger.kicad_sch (KiCad schematic)
At the start: 21 parts, among them U10 BQ25887RGER, U18 LM1084RS-5.0

Commit message: i finished and getting it made
Parts:
- removed U18: LM1084RS-5.0, Package_TO_SOT_SMD:TO-252-3_TabPin2, symbol Batt_Charger:LM1084RS-5.0
Connections:
- net VOUT is gone; now on net BAT_CHARGER_VIN: C18.2, L4.2 (A), TP11.1 (PAD), U10.23 (VBUS)
Changed lines of the file:
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@@
-	)
-	(junction
-		(at 180.34 73.66)
-		(diameter 0)
-		(color 0 0 0 0)
 	)
 	(junction
@@
 	(wire
 		(pts
-			(xy 189.23 76.2) (xy 189.23 73.66)
-		)
-		(stroke
-			(width 0)
-			(type default)
-		)
-	)
-	(wire
-		(pts
 			(xy 179.07 97.79) (xy 175.26 97.79)
 		)
@@
 	(wire
 		(pts
-			(xy 180.34 73.66) (xy 189.23 73.66)
-		)
-		(stroke
-			(width 0)
-			(type default)
-		)
-	)
-	(wire
-		(pts
 			(xy 187.96 78.74) (xy 187.96 76.2)
 		)
@@
 	(wire
 		(pts
-			(xy 189.23 78.74) (xy 187.96 78.74)
+			(xy 187.96 78.74) (xy 194.31 78.74)
 		)
 		(stroke
@@
 	(hierarchical_label "BAT_CHARGER_VIN"
 		(shape input)
-		(at 204.47 77.47 0)
+		(at 194.31 78.74 0)
 		(effects
 			(font
@@
 					(unit 1)
 				)
-			)
-		)
-	)
-	(symbol
-		(lib_id "Batt_Charger:LM1084RS-5.0")
-		(at 196.85 77.47 0)
-		(unit 1)
-		(body_style 1)
-		(exclude_from_sim no)
-		(in_bom yes)
-		(on_board yes)
-		(in_pos_files yes)
-		(dnp no)
-		(property "Reference" "U18"
-			(at 196.85 72.39 0)
-			(show_name no)
-			(do_not_autoplace no)
-			(effects
-				(font
-					(size 1.27 1.27)
-				)
-			)
-		)
-		(property "Value" "LM1084RS-5.0"
-			(at 196.85 70.358 0)
-			(show_name no)
-			(do_not_autoplace no)
-			(effects
-				(font
-					(size 1.27 1.27)
-				)
-			)
-		)
-		(property "Footprint" "Package_TO_SOT_SMD:TO-252-3_TabPin2"
-			(at 196.85 77.47 0)
-			(hide yes)
-			(show_name no)
-			(do_not_autoplace no)
-			(effects
-				(font
-					(size 1.27 1.27)
-				)
-			)
-		)
-		(property "Datasheet" ""
-			(at 196.85 77.47 0)
-			(hide yes)
-			(show_name no)
-			(do_not_autoplace no)
-			(effects
-				(font
-					(size 1.27 1.27)
-				)
-			)
-		)
-		(property "Description" ""
-			(at 196.85 77.47 0)
-			(hide yes)
-			(show_name no)
-			(do_not_autoplace no)
-			(effects
-				(font
-					(size 1.27 1.27)
-				)
-			)
-		)
-		(pin "1"
-		)
-		(pin "2"
-		)
-		(pin "3"
-		)
-		(instances
-			(project "PowerBox_PCB"
-				(path "/b0254e12-8cc0-427f-8cea-8f6ec8f66525/da3152ce-e99b-41cb-8d30-a5dc30414d8e"
-					(reference "U18")
-					(unit 1)
-				)
